File: PCB/acoustic_levitation_main.sch (KiCad schematic (older format))
At the start: 5 parts, among them J1 DE0-Nano-SoC: GPIO 0, J2 DE0-Nano-SoC: GPIO 1, J3 DE0-Nano-SoC: JP3, J4 DE0-Nano-SoC: JP2, J5 DE0-Nano-SoC: JP5[3]

Commit message: added output and rtc controll
Parts:
- J1, J2: symbol Conn_02x20_Odd_Even -> acoustic_levitation_main-rescue:Conn_02x20_Odd_Even
- J3: symbol Conn_01x08 -> acoustic_levitation_main-rescue:Conn_01x08
- J4: symbol Conn_01x10 -> acoustic_levitation_main-rescue:Conn_01x10
- J5: symbol Conn_01x01 -> acoustic_levitation_main-rescue:Conn_01x01
Connections:
- wire segments 125 -> 133
