File: PCB/conn_x14.sch (KiCad schematic (older format))
At the start: 1 part, among them J6 8-215079-8

Commit message: added output and rtc controll
Parts:
- J6: symbol Conn_02x09_Odd_Even -> acoustic_levitation_main-rescue:Conn_02x09_Odd_Even
Changed lines of the file:
@@
-EESchema Schematic File Version 2
-LIBS:power
-LIBS:device
-LIBS:switches
-LIBS:relays
-LIBS:motors
-LIBS:transistors
-LIBS:conn
-LIBS:linear
-LIBS:regul
-LIBS:74xx
-LIBS:cmos4000
-LIBS:adc-dac
-LIBS:memory
-LIBS:xilinx
-LIBS:microcontrollers
-LIBS:dsp
-LIBS:microchip
-LIBS:analog_switches
-LIBS:motorola
-LIBS:texas
-LIBS:intel
-LIBS:audio
-LIBS:interface
-LIBS:digital-audio
-LIBS:philips
-LIBS:display
-LIBS:cypress
-LIBS:siliconi
-LIBS:opto
-LIBS:atmel
-LIBS:contrib
-LIBS:valves
-LIBS:library
+EESchema Schematic File Version 4
 LIBS:acoustic_levitation_main-cache
-EELAYER 25 0
+EELAYER 29 0
 EELAYER END
 $Descr A4 11693 8268
 encoding utf-8
-Sheet 11 12
+Sheet 8 12
 Title "Acoustic levitation"
 Date "2018-03-24"
@@
 $EndDescr
 $Comp
-L Conn_02x09_Odd_Even J6
+L acoustic_levitation_main-rescue:Conn_02x09_Odd_Even J6
 U 1 1 5AAB02F6
 P 5800 3600
@@
 AR Path="/5AAAA010/5AAB02F6" Ref="J8"  Part="1"
 AR Path="/5AAAA0A0/5AAB02F6" Ref="J9"  Part="1"
-F 0 "J9" H 5850 4100 50  0000 C CNN
+F 0 "J6" H 5850 4100 50  0000 C CNN
 F 1 "8-215079-8" H 5750 3100 50  0000 L CNN
 F 2 "footprints:TE_8-215079-8" H 5800 3600 50  0001 C CNN
@@
 	5600 3800 5250 3800
 Wire Bus Line
-	6550 3000 6550 3700
-Wire Bus Line
 	4950 3000 6550 3000
-Wire Bus Line
-	5150 3000 5150 3700
 Text Label 6200 3800 0    60   ~ 0
 In14
@@
 	5500 4000 5500 4100
 $Comp
-L GND #PWR052
+L acoustic_levitation_main-rescue:GND #PWR052
 U 1 1 5AAA94F7
 P 5500 4100
@@
 AR Path="/5AAAA010/5AAA94F7" Ref="#PWR058"  Part="1"
 AR Path="/5AAAA0A0/5AAA94F7" Ref="#PWR061"  Part="1"
-F 0 "#PWR061" H 5500 3850 50  0001 C CNN
+F 0 "#PWR052" H 5500 3850 50  0001 C CNN
 F 1 "GND" H 5500 3950 50  0000 C CNN
 F 2 "" H 5500 4100 50  0001 C CNN
@@
 $EndComp
 $Comp
-L +3V3 #PWR053
+L acoustic_levitation_main-rescue:+3V3 #PWR053
 U 1 1 5AAA954A
 P 6450 4000
@@
 AR Path="/5AAAA010/5AAA954A" Ref="#PWR059"  Part="1"
 AR Path="/5AAAA0A0/5AAA954A" Ref="#PWR062"  Part="1"
-F 0 "#PWR062" H 6450 3850 50  0001 C CNN
+F 0 "#PWR053" H 6450 3850 50  0001 C CNN
 F 1 "+3V3" V 6450 4140 50  0000 L CNN
 F 2 "" H 6450 4000 50  0001 C CNN
@@
 $EndComp
 $Comp
-L +12V #PWR054
+L acoustic_levitation_main-rescue:+12V #PWR054
 U 1 1 5AAA9573
 P 6450 3900
@@
 AR Path="/5AAAA010/5AAA9573" Ref="#PWR060"  Part="1"
 AR Path="/5AAAA0A0/5AAA9573" Ref="#PWR063"  Part="1"
-F 0 "#PWR063" H 6450 3750 50  0001 C CNN
+AR Path="/5AAA9573" Ref="#PWR063"  Part="1"
+F 0 "#PWR054" H 6450 3750 50  0001 C CNN
 F 1 "+12V" V 6450 4040 50  0000 L CNN
 F 2 "" H 6450 3900 50  0001 C CNN
@@
 Wire Wire Line
 	6100 4000 6450 4000
+Wire Bus Line
+	6550 3000 6550 3700
+Wire Bus Line
+	5150 3000 5150 3700
 $EndSCHEMATC
